Commit message: add: obstacle model in rviz

File: src/lane_change_control/urdf/robot.urdf (robot description, URDF)
Before this commit: robot simple_robot, 6 links, 5 joints
Links:
- added link obstacle; visual box size=0.5 0.5 1.0
Joints:
- added joint obstacle_joint: type fixed, parent base_link, child obstacle, origin xyz=1.5 0 0.5 rpy=0 0 0

Commit message: fix: Kinect orient

File: src/lane_change_control/urdf/robot.urdf (robot description, URDF)
Before this commit: robot simple_robot, 7 links, 6 joints
Joints:
- joint camera_joint: origin xyz=0.25 0 0.2 rpy=-1.5708 0 -1.5708 -> xyz=0.25 0 0.2 rpy=0 0 0

Commit message: refractor: coordinate setting

File: src/lane_change_control/urdf/robot.urdf (robot description, URDF)
Before this commit: robot simple_robot, 7 links, 6 joints
Links:
- link base_link: geometry visual box size=0.2 0.05 0.02; visual box size=0.5 0.3 0.1

Commit message: fix: model height

File: src/lane_change_control/urdf/robot.urdf (robot description, URDF)
Before this commit: robot simple_robot, 7 links, 6 joints
Links:
- link base_link: geometry collision box size=0.5 0.3 0.1; visual box size=0.2 0.05 0.02
- link front_left_wheel: geometry collision cylinder length=0.05 radius=0.1; visual cylinder length=0.05 radius=0.1
- link front_right_wheel: geometry collision cylinder length=0.05 radius=0.1; visual cylinder length=0.05 radius=0.1
- link rear_left_wheel: geometry collision cylinder length=0.05 radius=0.1; visual cylinder length=0.05 radius=0.1
- link rear_right_wheel: geometry collision cylinder length=0.05 radius=0.1; visual cylinder length=0.05 radius=0.1
Joints:
- joint front_left_wheel_joint: origin xyz=0.15 0.175 0 rpy=1.5708 0 0 -> xyz=0.15 0.175 0.1 rpy=1.5708 0 0
- joint front_right_wheel_joint: origin xyz=0.15 -0.175 0 rpy=1.5708 0 0 -> xyz=0.15 -0.175 0.1 rpy=1.5708 0 0
- joint obstacle_joint: origin xyz=1.5 0 0.5 rpy=0 0 0 -> xyz=1.5 0 0 rpy=0 0 0
- joint rear_left_wheel_joint: origin xyz=-0.15 0.175 0 rpy=1.5708 0 0 -> xyz=-0.15 0.175 0.1 rpy=1.5708 0 0
- joint rear_right_wheel_joint: origin xyz=-0.15 -0.175 0 rpy=1.5708 0 0 -> xyz=-0.15 -0.175 0.1 rpy=1.5708 0 0

Commit message: add: road model in rviz

File: src/lane_change_control/urdf/robot.urdf (robot description, URDF)
Before this commit: robot simple_robot, 7 links, 6 joints
Links:
- added link road_plane; visual box size=25.0 6.0 0.1
- link base_link: geometry visual box size=0.2 0.05 0.02; visual box size=0.5 0.3 0.1
- link front_left_wheel: geometry visual cylinder length=0.05 radius=0.1
- link front_right_wheel: geometry visual cylinder length=0.05 radius=0.1
- link rear_left_wheel: geometry visual cylinder length=0.05 radius=0.1
- link rear_right_wheel: geometry visual cylinder length=0.05 radius=0.1
Joints:
- added joint road_joint: type fixed, parent base_link, child road_plane, origin xyz=2.5 0 -0.05 rpy=0 0 0
- joint front_left_wheel_joint: origin xyz=0.15 0.175 0.1 rpy=1.5708 0 0 -> xyz=0.15 0.175 0 rpy=1.5708 0 0
- joint front_right_wheel_joint: origin xyz=0.15 -0.175 0.1 rpy=1.5708 0 0 -> xyz=0.15 -0.175 0 rpy=1.5708 0 0
- joint obstacle_joint: origin xyz=1.5 0 0 rpy=0 0 0 -> xyz=1.5 0 0.5 rpy=0 0 0
- joint rear_left_wheel_joint: origin xyz=-0.15 0.175 0.1 rpy=1.5708 0 0 -> xyz=-0.15 0.175 0 rpy=1.5708 0 0
- joint rear_right_wheel_joint: origin xyz=-0.15 -0.175 0.1 rpy=1.5708 0 0 -> xyz=-0.15 -0.175 0 rpy=1.5708 0 0

Commit message: fix: all models height in rviz

File: src/lane_change_control/urdf/robot.urdf (robot description, URDF)
Before this commit: robot simple_robot, 8 links, 7 joints
Joints:
- joint camera_joint: origin xyz=0.25 0 0.2 rpy=0 0 0 -> xyz=0.25 0 0.3 rpy=0 0 0
- joint front_left_wheel_joint: origin xyz=0.15 0.175 0 rpy=1.5708 0 0 -> xyz=0.15 0.175 0.1 rpy=1.5708 0 0
- joint front_right_wheel_joint: origin xyz=0.15 -0.175 0 rpy=1.5708 0 0 -> xyz=0.15 -0.175 0.1 rpy=1.5708 0 0
- joint obstacle_joint: origin xyz=1.5 0 0.5 rpy=0 0 0 -> xyz=1.5 0 0.6 rpy=0 0 0
- joint rear_left_wheel_joint: origin xyz=-0.15 0.175 0 rpy=1.5708 0 0 -> xyz=-0.15 0.175 0.1 rpy=1.5708 0 0
- joint rear_right_wheel_joint: origin xyz=-0.15 -0.175 0 rpy=1.5708 0 0 -> xyz=-0.15 -0.175 0.1 rpy=1.5708 0 0

Commit message: fix: obstacle height

File: src/lane_change_control/urdf/robot.urdf (robot description, URDF)
Before this commit: robot simple_robot, 8 links, 7 joints
Links:
- removed link road_plane
Joints:
- removed joint road_joint
- joint camera_joint: origin xyz=0.25 0 0.3 rpy=0 0 0 -> xyz=0.25 0 0.2 rpy=0 0 0
- joint front_left_wheel_joint: origin xyz=0.15 0.175 0.1 rpy=1.5708 0 0 -> xyz=0.15 0.175 0 rpy=1.5708 0 0
- joint front_right_wheel_joint: origin xyz=0.15 -0.175 0.1 rpy=1.5708 0 0 -> xyz=0.15 -0.175 0 rpy=1.5708 0 0
- joint obstacle_joint: origin xyz=1.5 0 0.6 rpy=0 0 0 -> xyz=1.5 0 0.45 rpy=0 0 0
- joint rear_left_wheel_joint: origin xyz=-0.15 0.175 0.1 rpy=1.5708 0 0 -> xyz=-0.15 0.175 0 rpy=1.5708 0 0
- joint rear_right_wheel_joint: origin xyz=-0.15 -0.175 0.1 rpy=1.5708 0 0 -> xyz=-0.15 -0.175 0 rpy=1.5708 0 0

Commit message: fix: obstacle height +

File: src/lane_change_control/urdf/robot.urdf (robot description, URDF)
Before this commit: robot simple_robot, 7 links, 6 joints
Joints:
- joint obstacle_joint: origin xyz=1.5 0 0.45 rpy=0 0 0 -> xyz=1.5 0 0.4 rpy=0 0 0

Commit message: chore: remove obstacle in rviz

File: src/lane_change_control/urdf/robot.urdf (robot description, URDF)
Before this commit: robot simple_robot, 7 links, 6 joints
Links:
- removed link obstacle
Joints:
- removed joint obstacle_joint
